Commit message: 添加了新的基于位姿注册的中央协调器，但是发现slam_toolbox的回环检测目前会产生副作用导致地图歪斜扭曲

File: turtlebot3_gazebo/urdf/turtlebot3_waffle_2.urdf.xacro (robot description, xacro)
@@ -3,4 +3,5 @@
   <xacro:include filename="$(find turtlebot3_description)/urdf/common_properties.xacro"/>
   <xacro:include filename="$(find turtlebot3_gazebo)/urdf/turtlebot3_waffle_2.gazebo.xacro"/>
+  <xacro:property name="prefix" value="" />
   <xacro:property name="r200_cam_rgb_px" value="0.005"/>
   <xacro:property name="r200_cam_rgb_py" value="0.018"/>
